File: PCB_Driver_DC_Motor/DC_Motor/DC_Motor.kicad_pcb (KiCad board)
At the start: 4 copper layers, 101.6 x 101.6 mm, 48 parts, among them J101 Conn_01x02, J102 Conn_01x04, J103 Conn_01x02, J104 Conn_01x02, Q101 IRF540N, Q102 IRF540N, Q103 IRF540N, Q104 IRF540N, U101 STM32F030K6Tx, U102 LM317_TO-220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

Commit message: Add files via upload
Other:
- copper layers 4 -> 2
Changed lines of the file:
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@@
 	(layers
 		(0 "F.Cu" jumper)
-		(4 "In1.Cu" signal)
-		(6 "In2.Cu" signal)
 		(2 "B.Cu" jumper)
 		(9 "F.Adhes" user "F.Adhesive")
@@
 			)
 			(layer "dielectric 1"
-				(type "prepreg")
-				(thickness 0.1)
-				(material "FR4")
-				(epsilon_r 4.5)
-				(loss_tangent 0.02)
-			)
-			(layer "In1.Cu"
-				(type "copper")
-				(thickness 0.035)
-			)
-			(layer "dielectric 2"
 				(type "core")
-				(thickness 1.24)
-				(material "FR4")
-				(epsilon_r 4.5)
-				(loss_tangent 0.02)
-			)
-			(layer "In2.Cu"
-				(type "copper")
-				(thickness 0.035)
-			)
-			(layer "dielectric 3"
-				(type "prepreg")
-				(thickness 0.1)
+				(thickness 1.51)
 				(material "FR4")
 				(epsilon_r 4.5)
@@
 		(grid_origin 80.81 133.82)
 		(pcbplotparams
-			(layerselection 0x00000000_00000000_55555555_5755f5ff)
+			(layerselection 0x00000000_00000000_55555555_5755f5f5)
 			(plot_on_all_layers_selection 0x00000000_00000000_00000000_00000000)
 			(disableapertmacros no)

Commit message: Add files via upload
Other:
- board text added: "OCTOBER 2025"
- board text added: "PROTO_DC_DRIVER"
- board text added: "R.CASAS"
Changed lines of the file:
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@@
+	)
+	(gr_rect
+		(start 155.74 103.848)
+		(end 179.362 116.04)
+		(stroke
+			(width 0.25)
+			(type solid)
+		)
+		(fill no)
+		(layer "F.SilkS")
 	)
 	(gr_rect
@@
 		(layer "User.2")
 	)
+	(gr_text "R.CASAS"
+		(at 163.106 111.214 0)
+		(layer "F.Cu")
+		(effects
+			(font
+				(size 1.5 1.5)
+				(thickness 0.25)
+				(bold yes)
+			)
+			(justify left bottom)
+		)
+	)
+	(gr_text "OCTOBER 2025"
+		(at 158.788 114.516 0)
+		(layer "F.Cu")
+		(effects
+			(font
+				(size 1.5 1.5)
+				(thickness 0.25)
+				(bold yes)
+			)
+			(justify left bottom)
+		)
+	)
+	(gr_text "PROTO_DC_DRIVER"
+		(at 157.01 107.658 0)
+		(layer "F.Cu")
+		(effects
+			(font
+				(size 1.5 1.5)
+				(thickness 0.25)
+				(bold yes)
+			)
+			(justify left bottom)
+		)
+	)
 	(segment
